File: Macwan_lab_2/Part-1/Schematic/xyz/xyz.sch (KiCad schematic (older format))
At the start: 39 parts, among them J10 PwrHdr3, J11 PwrHdr4, J12 PwrHdr5, J13 PwrHdr6, J2 PwrHdr1, J3 PwrHdr2, J4 Header9, J5 DB9, J6 HEADER2_0, SW1 SPST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

Commit message: Updates
Parts:
- removed U4: 74LS373, symbol 74xx:74LS373
- added C20, C21, C22, C23: 0.1uF, symbol Device:C_Small
- added C?: 27pF, symbol Device:C_Small
- added D: GREEN_LED, symbol Device:LED
- added Q: 2N2222, symbol Transistor_BJT:2N2222
- added R: 330, symbol Device:R
- added R: 1K, symbol Device:R
Connections:
- net A15: now also U2.3 (I2); no longer U2.2 (I1)
- net ALE: now also U3.11 (LE), C?.2; no longer U2.5 (I4)
- net GND: now also C20.1, C21.1, C22.1, C23.1, C?.1, Q.1 (E)
- net VCC: now also C20.2, C21.2, C22.2, C23.2, R.1
- net ~EA~: now also U2.5 (I4); no longer U2.6 (I5)
- net ~OE~_1: now also U2.13 (IO7); no longer U2.14 (IO6)
- net ~PSEN~: now also U2.4 (I3)
- net ~RD~: no longer U2.3 (I2)
- net P1.5: now reaches U1.5 (P1.4)
- net P1.5: now also R.1
- net P1.7: now reaches U1.8 (P1.7)
- net LE_1: no longer names the net of U2.19 (IO1)
- net LE_1: no longer U3.11 (LE)
- net LE_2: no longer names the net of U2.18 (IO2)
- new net: Q.2 (B), R.2
- new net: D.1 (K), Q.3 (C)
- new net: D.2 (A), R.2
- no-connect marks 0 -> 24
Other:
- note added: "Decoupling Capacitors connected with every chip"
- note added: "Power LED connected to 8051 GPIO"
- note removed: "Demultiplexed Output (Data)"
- note removed: "Latch Circuits"
- moved on the sheet: U2
